File: LFO2/LFO2.kicad_pcb (KiCad board)
At the start: 2 copper layers, 19.7 x 100.3 mm, 42 parts, among them Q1 2N3904, Q2 2N3904, Q3 2N3904, Q4 2N3904, U1 TL074

Commit message: Add files via upload
Parts:
- added CV1: PJ3001F, benjiaomodular:AudioJack_3.5mm, B.Cu at (78.1, 99.6)
- added CV2: PJ3001F, benjiaomodular:AudioJack_3.5mm, B.Cu at (68.6, 99.6)
- added D1: 1N4148W, Diode_SMD:D_SOD-123, F.Cu at (81.3, 105.9)
- added D2: 1N4148W, Diode_SMD:D_SOD-123, F.Cu at (65.4, 105.9)
- added R25: 10K, Resistor_SMD:R_0805_2012Metric_Pad1.20x1.40mm_HandSolder, F.Cu at (81.3, 67.1)
- added R26: 4K7, Resistor_SMD:R_0805_2012Metric_Pad1.20x1.40mm_HandSolder, F.Cu at (80.1, 70.5)
- added R27: 4K7, Resistor_SMD:R_0805_2012Metric_Pad1.20x1.40mm_HandSolder, F.Cu at (69.2, 51.4)
- added R28: 10K, Resistor_SMD:R_0805_2012Metric_Pad1.20x1.40mm_HandSolder, F.Cu at (70.2, 54.6)
- added R29: 1K, Resistor_SMD:R_0805_2012Metric_Pad1.20x1.40mm_HandSolder, F.Cu at (78.5, 87.8)
- added R30: 1K, Resistor_SMD:R_0805_2012Metric_Pad1.20x1.40mm_HandSolder, F.Cu at (80.4, 52.5)
- C1, C2: footprint Capacitors_SMD:C_0805_HandSoldering -> Capacitor_SMD:C_0805_2012Metric_Pad1.18x1.45mm_HandSolder
- C3, C4: footprint Capacitors_SMD:CP_Elec_5x5.8 -> Capacitor_SMD:CP_Elec_5x5.9
- D3, D4: footprint Eurocad:LED3mm -> eurocad-master:LED3mm
- H1: footprint Pin_Headers:Pin_Header_Straight_2x05_Pitch2.54mm -> Connector_PinHeader_2.54mm:PinHeader_2x05_P2.54mm_Vertical
- Q1, Q2, Q3, Q4: footprint TO_SOT_Packages_SMD:SOT-23_Handsoldering -> Package_TO_SOT_SMD:SOT-23
- R1, R10, R11, R12, R13, R14, R15, R16, R17, R18, R19, R2, R20, R21, R22, R23, R24, R3, R4, R5, R6, R7, R8, R9: footprint Resistors_SMD:R_0805_HandSoldering -> Resistor_SMD:R_0805_2012Metric_Pad1.20x1.40mm_HandSolder
- SQ1, SQ2, TRI1, TRI2: value PJ301M-12 -> PJ3001F; footprint Eurocad:PJ301M-12 -> benjiaomodular:AudioJack_3.5mm
- U1: footprint Housings_SOIC:SOIC-14_3.9x8.7mm_Pitch1.27mm -> Package_SO:SOIC-14_3.9x8.7mm_P1.27mm
- moved R10 27.9 mm to (65.9, 52.6)
- moved R16 25.0 mm to (68.3, 65.9)
- moved R12 24.9 mm to (65.9, 65.9), turned to -90 degrees
- moved U1 23.9 mm to (73.7, 64.4)
- moved C1 23.8 mm to (79.0, 67.1)
- moved C2 23.4 mm to (68.3, 61.7)
- moved R11 23.4 mm to (81.3, 61.7)
- moved R15 23.4 mm to (79.0, 61.7)
- moved R9 22.8 mm to (80.5, 56.6), turned to -90 degrees
- moved C3 21.5 mm to (68.3, 79.9), turned to 45 degrees
- moved C4 21.0 mm to (77.9, 79.9), turned to -135 degrees
- moved Q3 18.6 mm to (66.3, 56.8)
- moved H1 15.5 mm to (68.2, 95.2), turned to 90 degrees
- moved R6 14.7 mm to (65.9, 61.7), turned to 90 degrees
- moved R8 13.1 mm to (65.9, 50.4), turned to 180 degrees
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Connections:
- D3 pad 1: Net-(D3-Pad1) -> Net-(D3-K)
- D4 pad 1: Net-(D4-Pad1) -> Net-(D4-K)
- Q1 pad 1: GND -> Net-(Q1-B)
- Q1 pad 2: Net-(Q1-Pad2) -> GND
- Q1 pad 3: Net-(Q1-Pad3) -> Net-(Q1-C)
- Q2 pad 1: Net-(Q2-Pad1) -> Net-(Q2-B)
- Q2 pad 2: Net-(D3-Pad1) -> Net-(Q2-E)
- Q2 pad 3: Net-(Q2-Pad3) -> Net-(D3-K)
- Q3 pad 1: GND -> Net-(Q3-B)
- Q3 pad 2: Net-(Q3-Pad2) -> GND
- Q3 pad 3: Net-(Q3-Pad3) -> Net-(Q3-C)
- Q4 pad 1: Net-(Q4-Pad1) -> Net-(Q4-B)
- Q4 pad 2: Net-(D4-Pad1) -> Net-(Q4-E)
- Q4 pad 3: Net-(Q4-Pad3) -> Net-(D4-K)
- R10 pad 1: Net-(Q3-Pad3) -> Net-(Q3-B)
- R13 pad 1: Net-(Q2-Pad3) -> Net-(Q2-B)
- R14 pad 1: Net-(Q4-Pad3) -> Net-(Q4-B)
- R17 pad 1: Net-(Q2-Pad1) -> Net-(Q2-E)
- R18 pad 1: Net-(Q4-Pad1) -> Net-(Q4-E)
- R5 pad 2: Net-(Q1-Pad2) -> Net-(Q1-C)
- R6 pad 2: Net-(Q3-Pad2) -> Net-(Q3-C)
- R9 pad 1: Net-(Q1-Pad3) -> Net-(Q1-B)
- RV1 pad 1: +12V -> Net-(R30-Pad1)
- RV1 pad 3: GND -> +12V
- RV2 pad 1: +12V -> Net-(R29-Pad1)
- RV2 pad 3: GND -> +12V
Routing:
- net Net-(Q1-Pad3): track 60.2 -> 0.00 mm, vias 3 -> 0
- net Net-(D2-K): track 0.00 -> 54.3 mm, vias 0 -> 2
- net Net-(D1-K): track 0.00 -> 37.3 mm
- net Net-(R3-Pad1): track 8.05 -> 40.4 mm, vias 0 -> 1
- net Net-(R10-Pad2): track 61.6 -> 88.1 mm
- net Net-(R15-Pad2): track 59.9 -> 83.3 mm
- net Net-(Q1-B): track 0.00 -> 23.2 mm
- net Net-(U1C--): track 38.8 -> 18.5 mm, vias 2 -> 0
- net +12V: track 80.9 -> 65.2 mm
- net Net-(U1A--): track 45.2 -> 32.2 mm
- net Net-(U1C-+): track 34.1 -> 21.7 mm
- net Net-(Q1-Pad2): track 12.2 -> 0.00 mm
- net Net-(Q3-Pad3): track 11.6 -> 0.00 mm
- net -12V: track 25.6 -> 36.0 mm, vias 2 -> 0
- net Net-(U1A-+): track 45.8 -> 37.6 mm, vias 2 -> 0
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Other:
- net class Default removed
